File: Punainen Husse.kicad_pcb (KiCad board)
At the start: 2 copper layers, 99.7 x 77.1 mm, 87 parts, among them Q1 MMBF4393LT1G, Q2 BC807, Q3 MMBF170, Q4 MMBF170, SW1 SW_DPDT_x2, SW2 SW_DPDT_x2, U1 TL074, U2 LF351D, U3 LM13700

Commit message: small fixes
Parts:
- removed ? (x12): , 
- removed Attack, Intensity: a1M, Potentiometer_THT:UT right angle long pin
- removed Level: a10k, Potentiometer_THT:UT right angle long pin
- removed REF**: Pin_D0.7mm_L6.5mm_W1.8mm_FlatFork, Connector_Pin:Pin_D0.7mm_L6.5mm_W1.8mm_FlatFork
- removed Ratio, Volume: a100k, Potentiometer_THT:UT right angle long pin
- removed Tone: b100k, Potentiometer_THT:UT right angle long pin
- added Rv1: a1M, Potentiometer_THT:UT right angle long pin, B.Cu at (199.0, 81.2)
- added Rv2: b100k, Potentiometer_THT:UT right angle long pin, B.Cu at (172.4, 99.3)
- added Rv3: a100k, Potentiometer_THT:UT right angle long pin, B.Cu at (171.0, 81.2)
- added Rv4: a100k, Potentiometer_THT:UT right angle long pin, B.Cu at (141.5, 99.2)
- added Rv5: a1M, Potentiometer_THT:UT right angle long pin, B.Cu at (143.0, 81.2)
- added Rv6: a10k, Potentiometer_THT:UT right angle long pin, B.Cu at (115.0, 81.2)
- added TP1: OUT, TestPoint:TestPoint_THTPad_D2.5mm_Drill1.2mm, F.Cu at (174.0, 129.0)
- added TP10: In_E, TestPoint:TestPoint_THTPad_D2.5mm_Drill1.2mm, F.Cu at (110.0, 116.0)
- added TP11: GND, TestPoint:TestPoint_THTPad_D2.5mm_Drill1.2mm, F.Cu at (181.4, 64.1)
- added TP12: 9V IN, TestPoint:TestPoint_THTPad_D2.5mm_Drill1.2mm, F.Cu at (188.6, 64.1)
- added TP2: IN, TestPoint:TestPoint_THTPad_D2.5mm_Drill1.2mm, F.Cu at (131.0, 129.0)
- added TP3: GND, TestPoint:TestPoint_THTPad_D2.5mm_Drill1.2mm, F.Cu at (137.0, 129.0)
- added TP4: GND, TestPoint:TestPoint_THTPad_D2.5mm_Drill1.2mm, F.Cu at (179.0, 129.0)
- added TP5: Out_R, TestPoint:TestPoint_THTPad_D2.5mm_Drill1.2mm, F.Cu at (185.0, 116.0)
- added TP6: In_R, TestPoint:TestPoint_THTPad_D2.5mm_Drill1.2mm, F.Cu at (179.0, 116.0)
- added TP7: R_FS, TestPoint:TestPoint_THTPad_D2.5mm_Drill1.2mm, F.Cu at (191.0, 116.0)
- added TP8: E_FS, TestPoint:TestPoint_THTPad_D2.5mm_Drill1.2mm, F.Cu at (123.0, 116.0)
- added TP9: Out_E, TestPoint:TestPoint_THTPad_D2.5mm_Drill1.2mm, F.Cu at (130.0, 116.0)
- moved C15 4.69 mm to (111.7, 71.6), turned to 180 degrees
Routing:
- net Net-(C9-Pad1): track 69.0 -> 63.9 mm
- net Net-(C15-Pad1): track 4.45 -> 6.98 mm
- net Net-(U1B-+): track 27.2 -> 28.4 mm
- net Net-(C15-Pad2): track 8.59 -> 9.55 mm
- net GND: vias 32 -> 33
Other:
- outline, holes or cut-outs redrawn
- board text removed: "{ "ViaStitching": "0.2", "stitch_zone_0": { "HSpacing": "1.27", "VSpacing": "1.27", "Clearance": "0.2", "Randomize": false } }"
