File: Punainen Husse.kicad_sch (KiCad schematic)
At the start: 75 parts, among them J1 Barrel_Jack_Switch, Q1 MMBF4393LT1G, Q2 MMBF170, Q3 MMBF170, Q4 BC807, SW1 SW_DPDT_x2, SW2 SW_DPDT_x2, U1 LF351D, U2 TL074, U3 LM13700

Commit message: small fixes
Parts:
- removed J1: Barrel_Jack_Switch, Connector_BarrelJack:BarrelJack_Horizontal, symbol Connector:Barrel_Jack_Switch
- added TP1: OUT, TestPoint:TestPoint_THTPad_D2.5mm_Drill1.2mm, symbol Connector:TestPoint
- added TP10: In_E, TestPoint:TestPoint_THTPad_D2.5mm_Drill1.2mm, symbol Connector:TestPoint
- added TP11, TP3, TP4: GND, TestPoint:TestPoint_THTPad_D2.5mm_Drill1.2mm, symbol Connector:TestPoint
- added TP12: 9V IN, TestPoint:TestPoint_THTPad_D2.5mm_Drill1.2mm, symbol Connector:TestPoint
- added TP2: IN, TestPoint:TestPoint_THTPad_D2.5mm_Drill1.2mm, symbol Connector:TestPoint
- added TP5: Out_R, TestPoint:TestPoint_THTPad_D2.5mm_Drill1.2mm, symbol Connector:TestPoint
- added TP6: In_R, TestPoint:TestPoint_THTPad_D2.5mm_Drill1.2mm, symbol Connector:TestPoint
- added TP7: R_FS, TestPoint:TestPoint_THTPad_D2.5mm_Drill1.2mm, symbol Connector:TestPoint
- added TP8: E_FS, TestPoint:TestPoint_THTPad_D2.5mm_Drill1.2mm, symbol Connector:TestPoint
- added TP9: Out_E, TestPoint:TestPoint_THTPad_D2.5mm_Drill1.2mm, symbol Connector:TestPoint
- Rv1: renamed from Intensity1; Kenttä4 (none) -> Intensity
- Rv2: renamed from Tone1; Kenttä4 (none) -> Tone
- Rv3: renamed from Volume1; Kenttä4 (none) -> Volume
- Rv4: renamed from Ratio1; Kenttä4 (none) -> Attack
- Rv5: renamed from Attack1; Kenttä4 (none) -> Ratio
- Rv6: renamed from Level1; Kenttä4 (none) -> Volume
Connections:
- net FS_engi: now also TP8.1
- net FS_red: now also TP7.1
- net GND: now also TP11.1, TP3.1, TP4.1
- net IN_engi: now also TP2.1
- net IN_engi_pcb: now also TP10.1
- net IN_red_pcb: now also TP6.1
- net OUT_engi_pcb: now also TP9.1
- net OUT_red: now also TP1.1
- net OUT_red_pcb: now also TP5.1
- net at R9.1: now also TP12.1
- no-connect marks 6 -> 5
Other:
- moved on the sheet: SW2B

Commit message: Rev 2
Parts:
- C3: LCSC# C376859 -> C94121
Changed lines of the file:
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@@
       (effects (font (size 1.27 1.27)) hide)
     )
-    (property "LCSC#" "C376859" (at 38.1 55.88 0)
+    (property "LCSC#" "C94121" (at 38.1 55.88 0)
       (effects (font (size 1.27 1.27)) hide)
     )

Commit message: Revision 2
Parts:
- removed C11: 10nF, Capacitor_SMD:C_0805_2012Metric_Pad1.18x1.45mm_HandSolder, symbol Device:C_Small
- removed R22: 220Ω, Resistor_SMD:R_0805_2012Metric_Pad1.20x1.40mm_HandSolder, symbol Device:R_Small
- removed R4: 1.8k, Resistor_SMD:R_0805_2012Metric_Pad1.20x1.40mm_HandSolder, symbol Device:R_Small
- removed R6: 2.2k, Resistor_SMD:R_0805_2012Metric_Pad1.20x1.40mm_HandSolder, symbol Device:R_Small
- removed TP10: In_E, TestPoint:TestPoint_THTPad_D2.5mm_Drill1.2mm, symbol Connector:TestPoint
- removed TP5: Out_R, TestPoint:TestPoint_THTPad_D2.5mm_Drill1.2mm, symbol Connector:TestPoint
- removed TP6: In_R, TestPoint:TestPoint_THTPad_D2.5mm_Drill1.2mm, symbol Connector:TestPoint
- removed TP7: R_FS, TestPoint:TestPoint_THTPad_D2.5mm_Drill1.2mm, symbol Connector:TestPoint
- removed TP8: E_FS, TestPoint:TestPoint_THTPad_D2.5mm_Drill1.2mm, symbol Connector:TestPoint
- removed TP9: Out_E, TestPoint:TestPoint_THTPad_D2.5mm_Drill1.2mm, symbol Connector:TestPoint
- removed U1: LF351D, Package_SO:SO-8_3.9x4.9mm_P1.27mm, symbol Amplifier_Operational:LF351D
- removed U2: TL074, Package_SO:SO-14_3.9x8.65mm_P1.27mm, symbol Amplifier_Operational:TL074
- added C11 (x2): 10nF, Capacitor_SMD:C_0805_2012Metric_Pad1.18x1.45mm_HandSolder, symbol Device:C_Small
- added R11 (x2): 4.7k, Resistor_SMD:R_0805_2012Metric_Pad1.20x1.40mm_HandSolder, symbol Device:R_Small
- added R23 (x2): 1k, Resistor_SMD:R_0805_2012Metric_Pad1.20x1.40mm_HandSolder, symbol Device:R_Small
- added R25 (x2): 100Ω, Resistor_SMD:R_0805_2012Metric_Pad1.20x1.40mm_HandSolder, symbol Device:R_Small
- added R8 (x2): 10k, Resistor_SMD:R_0805_2012Metric_Pad1.20x1.40mm_HandSolder, symbol Device:R_Small
- added U1, U2, U3: TL072, Package_SO:SO-8_3.9x4.9mm_P1.27mm, symbol Amplifier_Operational:TL072
- D1: footprint Diode_SMD:D_SOD-123F -> Diode_SMD:D_SOD-123
- TP1, TP11, TP12, TP2, TP3, TP4: footprint TestPoint:TestPoint_THTPad_D2.5mm_Drill1.2mm -> TestPoint:TestPoint_Pad_4.0x4.0mm
Connections:
- net +5V: now also R25.2, U1.6 (-), U1.7
- net +9V: now also C11.1, C11.1, R8.1, U1.8 (V+), U2.8 (V+), U3.8 (V+)
- net GND: now also C11.2, C11.2, R8.2, U1.4 (V-), U2.4 (V-), U3.4 (V-)
- net at D6.2 (A), Q4.1 (B): now also U1.1
- net at D6.1 (K), Q4.2 (E), R28.2: now also U1.2 (-)
- net at Rv2.1: now also R11.2, R11.2
- net at C6.1, C7.2: now also R11.1, R11.1
- net at C5.2, LED1.2 (A), LED2.1 (K)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: now also U2.7
- net at C13.2, R14.2, R15.1: now also U1.5 (+)
- net at LED1.1 (K), LED2.2 (A), R5.2: now also R23.2, U2.6 (-)
- net 9V in: now reaches R9.1, TP12.1
- net at C4.1: now also R23.2
- net at C19.1, R26.2: now also U1.3 (+)
- net at C15.2, R19.2, R20.2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: now also U3.6 (-)
- net at C14.1, R18.2: now also U3.3 (+), U3.5 (+)
- net at C15.1, R21.2, R23.1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: now also U3.7
- net at D4.1 (K), R24.2: now also U3.2 (-)
- net at D4.2 (A), D5.1 (K): now also U3.1
- net at R21.1, U3.3 (+): now also R25.1
- net at C2.2, R1.2, R2.1: now also U2.5 (+)
- new net: R25.1, R25.2
- new net: R23.1, R23.1
- new net: U2.1, U2.2 (-)
- new net: R8.1, R8.2, U2.3 (+)
- no-connect marks 5 -> 3
Other:
- moved on the sheet: C10, C4, TP11, TP3, TP4
